Commit message: single dynamixel control

File: open_manipulator_x_description/gazebo/open_manipulator_x.gazebo_original.xacro (robot description, xacro)
@@ -30,5 +30,4 @@
   </xacro:macro>
   <xacro:Link reference="${prefix}link1"/>
-  <!--
   <xacro:Link reference="${prefix}link2"/>
   <xacro:Link reference="${prefix}link3"/>
@@ -40,7 +39,5 @@
     <material>Gazebo/Red</material>
   </gazebo>
--->
   <xacro:SimpleTransmission trans="${prefix}trans1" joint="${prefix}joint1" actuator="${prefix}actuator1" />
-  <!--
   <xacro:SimpleTransmission trans="${prefix}trans2" joint="${prefix}joint2" actuator="${prefix}actuator2" />
   <xacro:SimpleTransmission trans="${prefix}trans3" joint="${prefix}joint3" actuator="${prefix}actuator3" />
@@ -48,5 +45,4 @@
   <xacro:SimpleTransmission trans="${prefix}trans5" joint="${prefix}gripper_left_joint" actuator="${prefix}actuator5" />
   <xacro:SimpleTransmission trans="${prefix}trans6" joint="${prefix}gripper_right_joint" actuator="${prefix}actuator6" />
--->
   </xacro:macro>
 </robot>

File: open_manipulator_x_description/urdf/open_manipulator_x.urdf.xacro (robot description, xacro)
@@ -27,5 +27,5 @@
       </inertial>
     </link>
-    <joint name="${prefix}joint1" type="revolute">
+    <!--<joint name="${prefix}joint1" type="revolute">
       <parent link="${prefix}link1"/>
       <child link="${prefix}link2"/>
@@ -226,5 +226,5 @@
         <material name="red"/>
        </visual>
-    </link>
+    </link> -->
   </xacro:macro>
 </robot>

File: open_manipulator_x_description/urdf/open_manipulator_x_robot.urdf.xacro (robot description, xacro)
@@ -13,5 +13,9 @@
   <!-- Import URDF -->
   <xacro:include filename="$(find open_manipulator_x_description)/urdf/open_manipulator_x.urdf.xacro" />
+<!--
   <xacro:include filename="$(find open_manipulator_x_description)/ros2_control/open_manipulator_x_system.ros2_control.xacro" />
+  -->
+  <!--Added for the single motor effort control -->
+ <xacro:include filename="$(find open_manipulator_x_description)/ros2_control/testFile.ros2_control.xacro" />
   <xacro:open_manipulator_x prefix="$(arg prefix)" />
   <xacro:open_manipulator_x_gazebo prefix="$(arg prefix)" />
@@ -22,5 +26,5 @@
     port_name="$(arg port_name)"/>
   <gazebo>
-    <plugin name="gz_ros2_control::GazeboSimROS2ControlPlugin" filename="gz_ros2_control-system">
+   <plugin name="gz_ros2_control::GazeboSimROS2ControlPlugin" filename="gz_ros2_control-system">
       <parameters>$(find open_manipulator_x_bringup)/config/gz_controller_manager.yaml</parameters>
     </plugin>
